Commit message: fixed tof sensor issues

File: stochlite_champ/stochlite_description/urdf/stochlite.gazebo.xacro (robot description, xacro)
@@ -8,7 +8,7 @@
             </plugin>
         </gazebo>
-        <gazebo>
+        <!-- <gazebo>
             <self_collide>1</self_collide>
-        </gazebo>
+        </gazebo> -->
         <gazebo>
             <plugin filename="libgazebo_ros_p3d.so" name="p3d_base_controller">
@@ -23,54 +23,4 @@
             </plugin>
         </gazebo>
-        <gazebo>
-            <plugin filename="libhector_gazebo_ros_imu.so" name="imu_controller">
-                <updateRate>50.0</updateRate>
-                <bodyName>imu_link</bodyName>
-                <topicName>imu/data</topicName>
-                <accelDrift>0.005 0.005 0.005</accelDrift>
-                <accelGaussianNoise>0.005 0.005 0.005</accelGaussianNoise>
-                <rateDrift>0.005 0.005 0.005 </rateDrift>
-                <rateGaussianNoise>0.005 0.005 0.005 </rateGaussianNoise>
-                <headingDrift>0.005</headingDrift>
-                <headingGaussianNoise>0.005</headingGaussianNoise>
-            </plugin>
-        </gazebo>
-        <gazebo reference="tof_link">
-            <sensor type="ray" name="tof_sensor">
-                <visualize>true</visualize>
-                <update_rate>70</update_rate>
-                <always_on>1</always_on>
-                <ray>
-                    <scan>
-                        <horizontal>
-                            <samples>10</samples>
-                            <resolution>2</resolution>
-                            <min_angle>-0.02618</min_angle>
-                            <max_angle>0.02618</max_angle>
-                        </horizontal>
-                        <vertical>
-                            <samples>10</samples>
-                            <resolution>2</resolution>
-                            <min_angle>-0.02618</min_angle>
-                            <max_angle>0.02618</max_angle>
-                        </vertical>
-                    </scan>
-                    <range>
-                        <min>0.02</min>
-                        <max>2</max>
-                        <!-- <radius>0.33974388395</radius> -->
-                        <resolution>0.05</resolution>
-                    </range>
-                </ray>
-                <plugin name="tof_plugin" filename="libgazebo_ros_range.so">
-                    <topicName>gazebo/range_tof</topicName>
-                    <frameName>range_tof_map</frameName>
-                    <gaussianNoise>0.06</gaussianNoise>
-                    <updateRate>70</updateRate>
-                    <radiation>light</radiation>
-                    <fov>0.43</fov>
-                </plugin>
-            </sensor>
-        </gazebo>
     </xacro:macro>
 </robot>

File: stochlite_champ/stochlite_description/urdf/stochlite.materials.xacro (robot description, xacro)
@@ -1,6 +1,15 @@
 <?xml version="1.0"?>
 <robot xmlns:xacro="http://www.ros.org/wiki/xacro">
-    <xacro:macro name="stochlite_materials">
-        <!-- Add material and friction -->
+    <xacro:macro name="stochlite_materials" params="name color">
+        <gazebo reference="${name}_link">
+            <material>Gazebo/${color}</material>
+            <kp>10000000.0</kp>
+            <kd>1.0</kd>
+            <mu1>4.0</mu1>
+            <mu2>4.0</mu2>
+            <maxVel>0.0</maxVel>
+            <minDepth>0.001</minDepth>
+        </gazebo>
+        <!--
         <gazebo reference="base_link_torso">
             <material>Gazebo/White</material>
@@ -119,11 +128,5 @@
             <maxVel>0.0</maxVel>
             <minDepth>0.001</minDepth>
-        </gazebo>
-        <gazebo reference="tof_link">
-            <material>Gazebo/Red</material>
-        </gazebo>
-        <gazebo reference="imu_link">
-            <material>Gazebo/Yellow</material>
-        </gazebo>
+        </gazebo> -->
     </xacro:macro>
 </robot>

File: stochlite_champ/stochlite_description/urdf/stochlite.sensors.xacro (robot description, xacro)
@@ -1,6 +1,6 @@
 <?xml version="1.0"?>
 <robot xmlns:xacro="http://www.ros.org/wiki/xacro">
-    <xacro:macro name="stochlite_sensors">
-        <link name="imu_link">
+    <xacro:macro name="imu" params="id x y z roll pitch yaw update_rate">
+        <link name="imu_link_${id}">
             <inertial>
                 <mass value="0.001"/>
@@ -11,5 +11,4 @@
                 <origin xyz="0 0 0" rpy="0 0 0"/>
                 <geometry>
-                    <!-- <mesh filename="package://stochlite_description/meshes/VL53L0X.STL"/> -->
                     <box size="0.005 0.005 0.005" />
                 </geometry>
@@ -19,11 +18,27 @@
             </visual>
         </link>
-        <joint name="imu_joint" type="fixed">
+        <joint name="imu_joint_${id}" type="fixed">
             <parent link="base_link"/>
-            <child link="imu_link"/>
-            <origin xyz="0 0 0.005" rpy="0 0 0"/>
+            <child link="imu_link_${id}"/>
+            <origin xyz="${x} ${y} ${z}" rpy="${roll} ${pitch} ${yaw}"/>
         </joint>
+        <gazebo>
+            <plugin filename="libhector_gazebo_ros_imu.so" name="imu_${id}_controller">
+                <updateRate>${update_rate}</updateRate>
+                <bodyName>imu_link_${id}</bodyName>
+                <topicName>imu_${id}/data</topicName>
+                <accelDrift>0.005 0.005 0.005</accelDrift>
+                <accelGaussianNoise>0.005 0.005 0.005</accelGaussianNoise>
+                <rateDrift>0.005 0.005 0.005 </rateDrift>
+                <rateGaussianNoise>0.005 0.005 0.005 </rateGaussianNoise>
+                <headingDrift>0.005</headingDrift>
+                <headingGaussianNoise>0.005</headingGaussianNoise>
+            </plugin>
+            <material>Gazebo/Yellow</material>
+        </gazebo>
+    </xacro:macro>
+    <xacro:macro name='tof' params="id x y z roll pitch yaw update_rate">
         <!-- VL53L0X ToF sensor-->
-        <link name="tof_link">
+        <link name="tof_link_${id}">
             <inertial>
                 <mass value="0.001"/>
@@ -34,17 +49,54 @@
                 <origin xyz="0 0 0" rpy="0 0 0"/>
                 <geometry>
-                    <!-- <mesh filename="package://stochlite_description/meshes/VL53L0X.STL"/> -->
                     <box size="0.005 0.015 0.005" />
                 </geometry>
-                <material name="">
+                <material name="Red">
                     <color rgba="1 0.2 0.2 1" />
                 </material>
             </visual>
         </link>
-        <joint name="tof_joint" type="fixed">
-            <origin xyz="0 0 -0.029" rpy="0 1.57 0"/>
+        <joint name="tof_joint_${id}" type="fixed">
+            <origin xyz="${x} ${y} ${z}" rpy="${roll} ${pitch} ${yaw}"/>
+            <!-- <origin xyz="0 0 -0.029" rpy="0 1.57 0"/> -->
             <parent link="base_link"/>
-            <child link="tof_link"/>
+            <child link="tof_link_${id}"/>
         </joint>
+        <gazebo reference="tof_link_${id}">
+            <sensor type="ray" name="tof_sensor_${id}">
+                <visualize>true</visualize>
+                <update_rate>${update_rate}</update_rate>
+                <always_on>1</always_on>
+                <ray>
+                    <scan>
+                        <horizontal>
+                            <samples>10</samples>
+                            <resolution>1</resolution>
+                            <min_angle>-0.02618</min_angle>
+                            <max_angle>0.02618</max_angle>
+                        </horizontal>
+                        <vertical>
+                            <samples>10</samples>
+                            <resolution>1</resolution>
+                            <min_angle>-0.02618</min_angle>
+                            <max_angle>0.02618</max_angle>
+                        </vertical>
+                    </scan>
+                    <range>
+                        <min>0.002</min>
+                        <max>2</max>
+                        <resolution>0.005</resolution>
+                    </range>
+                </ray>
+                <plugin name="tof_plugin_${id}" filename="libgazebo_ros_range.so">
+                    <topicName>gazebo/range_tof_${id}</topicName>
+                    <frameName>frame_range_tof_${id}</frameName>
+                    <gaussianNoise>0.006</gaussianNoise>
+                    <updateRate>${update_rate}</updateRate>
+                    <radiation>light</radiation>
+                    <fov>0.43</fov>
+                </plugin>
+            </sensor>
+            <material>Gazebo/Red</material>
+        </gazebo>
     </xacro:macro>
 </robot>

File: stochlite_champ/stochlite_description/urdf/stochlite.transmission.xacro (robot description, xacro)
@@ -1,6 +1,15 @@
 <?xml version="1.0"?>
 <robot xmlns:xacro="http://www.ros.org/wiki/xacro">
-    <xacro:macro name="stochlite_transmission">
-        <transmission name="fl_abd_trans">
+    <xacro:macro name="stochlite_transmission" params="name">
+        <transmission name="${name}_trans">
+            <type>transmission_interface/SimpleTransmission</type>
+            <joint name="${name}_joint">
+                <hardwareInterface>hardware_interface/EffortJointInterface</hardwareInterface>
+            </joint>
+            <actuator name="${name}_motor">
+                <mechanicalReduction>1</mechanicalReduction>
+            </actuator>
+        </transmission>
+        <!-- <transmission name="fl_abd_trans">
             <type>transmission_interface/SimpleTransmission</type>
             <joint name="fl_abd_joint">
@@ -109,5 +118,5 @@
                 <mechanicalReduction>1</mechanicalReduction>
             </actuator>
-        </transmission>
+        </transmission> -->
     </xacro:macro>
 </robot>

File: stochlite_champ/stochlite_description/urdf/stochlite.urdf (robot description, URDF)
Before this commit: robot stochlite, 19 links, 18 joints
Links:
- removed link imu_link
- removed link tof_link
- added link imu_link_0, mass 0.001; visual box size=0.005 0.005 0.005
- added link tof_link_0, mass 0.001; visual box size=0.005 0.015 0.005
- added link tof_link_1, mass 0.001; visual box size=0.005 0.015 0.005
- added link tof_link_2, mass 0.001; visual box size=0.005 0.015 0.005
- added link tof_link_3, mass 0.001; visual box size=0.005 0.015 0.005
- added link tof_link_4, mass 0.001; visual box size=0.005 0.015 0.005
- added link tof_link_5, mass 0.001; visual box size=0.005 0.015 0.005
Joints:
- removed joint imu_joint
- removed joint tof_joint
- added joint imu_joint_0: type fixed, parent base_link, child imu_link_0, origin xyz=0.0 0.0 0.005 rpy=0.0 0.0 0.0
- added joint tof_joint_0: type fixed, parent base_link, child tof_link_0, origin xyz=0.15 0.0 -0.025 rpy=0.0 1.57 0.0
- added joint tof_joint_1: type fixed, parent base_link, child tof_link_1, origin xyz=0.065 0.047 -0.025 rpy=0.0 1.57 0.0
- added joint tof_joint_2: type fixed, parent base_link, child tof_link_2, origin xyz=0.065 -0.047 -0.025 rpy=0.0 1.57 0.0
- added joint tof_joint_3: type fixed, parent base_link, child tof_link_3, origin xyz=-0.15 0.0 -0.025 rpy=0.0 1.57 0.0
- added joint tof_joint_4: type fixed, parent base_link, child tof_link_4, origin xyz=-0.065 0.047 -0.025 rpy=0.0 1.57 0.0
- added joint tof_joint_5: type fixed, parent base_link, child tof_link_5, origin xyz=-0.065 -0.047 -0.025 rpy=0.0 1.57 0.0

File: stochlite_champ/stochlite_description/urdf/stochlite.urdf.xacro (robot description, xacro)
@@ -8,10 +8,52 @@
     <!-- <xacro:include filename="$(find teraranger_description)/urdf/base_hub.urdf.xacro"/> -->
     <!-- <xacro:include filename="$(find teraranger_description)/urdf/teraranger_one.urdf.xacro"/>     -->
+    <!-- For defining the links and joints-->
     <xacro:stochlite_description />
-    <xacro:stochlite_sensors />
-    <!-- <xacro:base_hub multi_hub="0" hub_id="0" parent="base_link" x="0" y="0.000" z="-0.029" roll="0.0" pitch="0.0" yaw="0.0"/> -->
-    <!-- <xacro:teraranger_one multi_hub="0" hub_id="0" id="0" x="0" y="0.000" z="0.000" roll="0.0" pitch="1.57" yaw="0.0" gaussian_noise="0.06"/> -->
-    <xacro:stochlite_transmission />
+    <!-- For hardware interface and ros control-->
+    <xacro:stochlite_transmission name="fl_abd"/>
+    <xacro:stochlite_transmission name="fl_hip"/>
+    <xacro:stochlite_transmission name="fl_knee"/>
+    <xacro:stochlite_transmission name="bl_abd"/>
+    <xacro:stochlite_transmission name="bl_hip"/>
+    <xacro:stochlite_transmission name="bl_knee"/>
+    <xacro:stochlite_transmission name="fr_abd"/>
+    <xacro:stochlite_transmission name="fr_hip"/>
+    <xacro:stochlite_transmission name="fr_knee"/>
+    <xacro:stochlite_transmission name="br_abd"/>
+    <xacro:stochlite_transmission name="br_hip"/>
+    <xacro:stochlite_transmission name="br_knee"/>
+    <!-- Materials and friction properties-->
+    <xacro:stochlite_materials name="base_link" color="White"/>
+    <xacro:stochlite_materials name="fl_abd" color="Grey"/>
+    <xacro:stochlite_materials name="bl_abd" color="Grey"/>
+    <xacro:stochlite_materials name="fr_abd" color="Grey"/>
+    <xacro:stochlite_materials name="br_abd" color="Grey"/>
+    <xacro:stochlite_materials name="fl_thigh" color="DarkGrey"/>
+    <xacro:stochlite_materials name="bl_thigh" color="DarkGrey"/>
+    <xacro:stochlite_materials name="fr_thigh" color="DarkGrey"/>
+    <xacro:stochlite_materials name="br_thigh" color="DarkGrey"/>
+    <xacro:stochlite_materials name="fl_shank" color="Grey"/>
+    <xacro:stochlite_materials name="bl_shank" color="Grey"/>
+    <xacro:stochlite_materials name="fr_shank" color="Grey"/>
+    <xacro:stochlite_materials name="br_shank" color="Grey"/>
+    <!-- For miscellaneous gazebo properties like ros-control etc. -->
     <xacro:stochlite_gazebo />
-    <xacro:stochlite_materials />
+    <!-- For sensors-->
+    <xacro:imu id="0" x="0.0" y="0.0" z="0.005" roll="0.0" pitch="0.0" yaw="0.0" update_rate="100"/>
+    <!-- front triangle of tofs -->
+    <xacro:tof id="0" x="0.150" y=" 0.000" z="-0.025" roll="0.0" pitch="1.57" yaw="0.0" update_rate="20"/>
+    <xacro:tof id="1" x="0.065" y=" 0.047" z="-0.025" roll="0.0" pitch="1.57" yaw="0.0" update_rate="20"/>
+    <xacro:tof id="2" x="0.065" y="-0.047" z="-0.025" roll="0.0" pitch="1.57" yaw="0.0" update_rate="20"/>
+    <!-- back triangle of tofs -->
+    <xacro:tof id="3" x="-0.150" y=" 0.000" z="-0.025" roll="0.0" pitch="1.57" yaw="0.0" update_rate="20"/>
+    <xacro:tof id="4" x="-0.065" y=" 0.047" z="-0.025" roll="0.0" pitch="1.57" yaw="0.0" update_rate="20"/>
+    <xacro:tof id="5" x="-0.065" y="-0.047" z="-0.025" roll="0.0" pitch="1.57" yaw="0.0" update_rate="20"/>
+    <!-- front triangle of tofs -->
+    <!-- <xacro:tof id="0" x="0.16" y=" 0.00" z="-0.025" roll="0.0" pitch="1.57" yaw="0.0" update_rate="20"/>
+    <xacro:tof id="1" x="0.06" y=" 0.055" z="-0.025" roll="0.0" pitch="1.57" yaw="0.0" update_rate="20"/>
+    <xacro:tof id="2" x="0.06" y="-0.055" z="-0.025" roll="0.0" pitch="1.57" yaw="0.0" update_rate="20"/> -->
+    <!-- back triangle of tofs -->
+    <!-- <xacro:tof id="3" x="-0.16" y=" 0.00" z="-0.025" roll="0.0" pitch="1.57" yaw="0.0" update_rate="20"/>
+    <xacro:tof id="4" x="-0.06" y=" 0.055" z="-0.025" roll="0.0" pitch="1.57" yaw="0.0" update_rate="20"/>
+    <xacro:tof id="5" x="-0.06" y="-0.055" z="-0.025" roll="0.0" pitch="1.57" yaw="0.0" update_rate="20"/> -->
 </robot>
