Commit message: added slope estimation

File: stochlite_champ/stochlite_description/urdf/stochlite.urdf (robot description, URDF)
Before this commit: robot stochlite, 24 links, 23 joints
Links:
- removed link imu_link_0
- removed link tof_link_0
- added link imu_link_1, mass 0.001; visual box size=0.005 0.005 0.005
- added link tof_link_6, mass 0.001; visual box size=0.005 0.015 0.005
Joints:
- removed joint imu_joint_0
- removed joint tof_joint_0
- added joint imu_joint_1: type fixed, parent base_link, child imu_link_1, origin xyz=0.0 0.0 0.005 rpy=0.0 0.0 0.0
- added joint tof_joint_6: type fixed, parent base_link, child tof_link_6, origin xyz=0.065 -0.047 -0.025 rpy=0.0 1.57 0.0
- joint tof_joint_1: origin xyz=0.065 0.047 -0.025 rpy=0.0 1.57 0.0 -> xyz=0.15 0.0 -0.025 rpy=0.0 1.57 0.0
- joint tof_joint_2: origin xyz=0.065 -0.047 -0.025 rpy=0.0 1.57 0.0 -> xyz=0.065 0.047 -0.025 rpy=0.0 1.57 0.0
- joint tof_joint_3: origin xyz=-0.15 0.0 -0.025 rpy=0.0 1.57 0.0 -> xyz=-0.065 0.047 -0.025 rpy=0.0 1.57 0.0
- joint tof_joint_4: origin xyz=-0.065 0.047 -0.025 rpy=0.0 1.57 0.0 -> xyz=-0.15 0.0 -0.025 rpy=0.0 1.57 0.0

File: stochlite_champ/stochlite_description/urdf/stochlite.urdf.xacro (robot description, xacro)
@@ -40,12 +40,12 @@
     <xacro:stochlite_gazebo />
     <!-- For sensors-->
-    <xacro:imu id="0" x="0.0" y="0.0" z="0.005" roll="0.0" pitch="0.0" yaw="0.0" update_rate="100"/>
+    <xacro:imu id="1" x="0.0" y="0.0" z="0.005" roll="0.0" pitch="0.0" yaw="0.0" update_rate="20"/>
     <!-- front triangle of tofs -->
-    <xacro:tof id="0" x="0.150" y=" 0.000" z="-0.025" roll="0.0" pitch="1.57" yaw="0.0" update_rate="20"/>
-    <xacro:tof id="1" x="0.065" y=" 0.047" z="-0.025" roll="0.0" pitch="1.57" yaw="0.0" update_rate="20"/>
-    <xacro:tof id="2" x="0.065" y="-0.047" z="-0.025" roll="0.0" pitch="1.57" yaw="0.0" update_rate="20"/>
+    <xacro:tof id="1" x="0.150" y=" 0.000" z="-0.025" roll="0.0" pitch="1.57" yaw="0.0" update_rate="20"/>
+    <xacro:tof id="2" x="0.065" y=" 0.047" z="-0.025" roll="0.0" pitch="1.57" yaw="0.0" update_rate="20"/>
+    <xacro:tof id="6" x="0.065" y="-0.047" z="-0.025" roll="0.0" pitch="1.57" yaw="0.0" update_rate="20"/>
     <!-- back triangle of tofs -->
-    <xacro:tof id="3" x="-0.150" y=" 0.000" z="-0.025" roll="0.0" pitch="1.57" yaw="0.0" update_rate="20"/>
-    <xacro:tof id="4" x="-0.065" y=" 0.047" z="-0.025" roll="0.0" pitch="1.57" yaw="0.0" update_rate="20"/>
+    <xacro:tof id="4" x="-0.150" y=" 0.000" z="-0.025" roll="0.0" pitch="1.57" yaw="0.0" update_rate="20"/>
+    <xacro:tof id="3" x="-0.065" y=" 0.047" z="-0.025" roll="0.0" pitch="1.57" yaw="0.0" update_rate="20"/>
     <xacro:tof id="5" x="-0.065" y="-0.047" z="-0.025" roll="0.0" pitch="1.57" yaw="0.0" update_rate="20"/>
     <!-- front triangle of tofs -->
