Commit message: final changes to slope estimation and urdf

File: stochlite_champ/stochlite_description/urdf/stochlite.materials.xacro (robot description, xacro)
@@ -11,122 +11,4 @@
             <minDepth>0.001</minDepth>
         </gazebo>
-        <!--
-        <gazebo reference="base_link_torso">
-            <material>Gazebo/White</material>
-            <kp>10000000.0</kp>
-            <kd>1.0</kd>
-            <mu1>4.0</mu1>
-            <mu2>4.0</mu2>
-            <maxVel>0.0</maxVel>
-            <minDepth>0.001</minDepth>
-        </gazebo>
-        <gazebo reference="fl_abd_link">
-            <material>Gazebo/Grey</material>
-            <kp>10000000.0</kp>
-            <kd>1.0</kd>
-            <mu1>4.0</mu1>
-            <mu2>4.0</mu2>
-            <maxVel>0.0</maxVel>
-            <minDepth>0.001</minDepth>
-        </gazebo>
-        <gazebo reference="fl_thigh_link">
-            <material>Gazebo/DarkGrey</material>
-            <kp>10000000.0</kp>
-            <kd>1.0</kd>
-            <mu1>4.0</mu1>
-            <mu2>4.0</mu2>
-            <maxVel>0.0</maxVel>
-            <minDepth>0.001</minDepth>
-        </gazebo>
-        <gazebo reference="fl_shank_link">
-            <material>Gazebo/Grey</material>
-            <kp>10000000.0</kp>
-            <kd>1.0</kd>
-            <mu1>4.0</mu1>
-            <mu2>4.0</mu2>
-            <maxVel>0.0</maxVel>
-            <minDepth>0.001</minDepth>
-        </gazebo>
-        <gazebo reference="fr_abd_link">
-            <material>Gazebo/Grey</material>
-            <kp>10000000.0</kp>
-            <kd>1.0</kd>
-            <mu1>4.0</mu1>
-            <mu2>4.0</mu2>
-            <maxVel>0.0</maxVel>
-            <minDepth>0.001</minDepth>
-        </gazebo>
-        <gazebo reference="fr_thigh_link">
-            <material>Gazebo/DarkGrey</material>
-            <kp>10000000.0</kp>
-            <kd>1.0</kd>
-            <mu1>4.0</mu1>
-            <mu2>4.0</mu2>
-            <maxVel>0.0</maxVel>
-            <minDepth>0.001</minDepth>
-        </gazebo>
-        <gazebo reference="fr_shank_link">
-            <material>Gazebo/Grey</material>
-            <kp>10000000.0</kp>
-            <kd>1.0</kd>
-            <mu1>4.0</mu1>
-            <mu2>4.0</mu2>
-            <maxVel>0.0</maxVel>
-            <minDepth>0.001</minDepth>
-        </gazebo>
-        <gazebo reference="bl_abd_link">
-            <material>Gazebo/Grey</material>
-            <kp>10000000.0</kp>
-            <kd>1.0</kd>
-            <mu1>4.0</mu1>
-            <mu2>4.0</mu2>
-            <maxVel>0.0</maxVel>
-            <minDepth>0.001</minDepth>
-        </gazebo>
-        <gazebo reference="bl_thigh_link">
-            <material>Gazebo/DarkGrey</material>
-            <kp>10000000.0</kp>
-            <kd>1.0</kd>
-            <mu1>4.0</mu1>
-            <mu2>4.0</mu2>
-            <maxVel>0.0</maxVel>
-            <minDepth>0.001</minDepth>
-        </gazebo>
-        <gazebo reference="bl_shank_link">
-            <material>Gazebo/Grey</material>
-            <kp>10000000.0</kp>
-            <kd>1.0</kd>
-            <mu1>4.0</mu1>
-            <mu2>4.0</mu2>
-            <maxVel>0.0</maxVel>
-            <minDepth>0.001</minDepth>
-        </gazebo>
-        <gazebo reference="br_abd_link">
-            <material>Gazebo/Grey</material>
-            <kp>10000000.0</kp>
-            <kd>1.0</kd>
-            <mu1>4.0</mu1>
-            <mu2>4.0</mu2>
-            <maxVel>0.0</maxVel>
-            <minDepth>0.001</minDepth>
-        </gazebo>
-        <gazebo reference="br_thigh_link">
-            <material>Gazebo/DarkGrey</material>
-            <kp>10000000.0</kp>
-            <kd>1.0</kd>
-            <mu1>4.0</mu1>
-            <mu2>4.0</mu2>
-            <maxVel>0.0</maxVel>
-            <minDepth>0.001</minDepth>
-        </gazebo>
-        <gazebo reference="br_shank_link">
-            <material>Gazebo/Grey</material>
-            <kp>10000000.0</kp>
-            <kd>1.0</kd>
-            <mu1>4.0</mu1>
-            <mu2>4.0</mu2>
-            <maxVel>0.0</maxVel>
-            <minDepth>0.001</minDepth>
-        </gazebo> -->
     </xacro:macro>
 </robot>

File: stochlite_champ/stochlite_description/urdf/stochlite.sensors.xacro (robot description, xacro)
@@ -1,5 +1,5 @@
 <?xml version="1.0"?>
 <robot xmlns:xacro="http://www.ros.org/wiki/xacro">
-    <xacro:macro name="imu" params="id x y z roll pitch yaw update_rate">
+    <xacro:macro name="imu" params="id x y z roll pitch yaw update_rate gnoise">
         <link name="imu_link_${id}">
             <inertial>
@@ -29,14 +29,14 @@
                 <topicName>imu_${id}/data</topicName>
                 <accelDrift>0.005 0.005 0.005</accelDrift>
-                <accelGaussianNoise>0.005 0.005 0.005</accelGaussianNoise>
+                <accelGaussianNoise>${gnoise} ${gnoise} ${gnoise}</accelGaussianNoise>
                 <rateDrift>0.005 0.005 0.005 </rateDrift>
-                <rateGaussianNoise>0.005 0.005 0.005 </rateGaussianNoise>
+                <rateGaussianNoise>${gnoise} ${gnoise} ${gnoise}</rateGaussianNoise>
                 <headingDrift>0.005</headingDrift>
-                <headingGaussianNoise>0.005</headingGaussianNoise>
+                <headingGaussianNoise>${gnoise}</headingGaussianNoise>
             </plugin>
             <material>Gazebo/Yellow</material>
         </gazebo>
     </xacro:macro>
-    <xacro:macro name='tof' params="id x y z roll pitch yaw update_rate">
+    <xacro:macro name='tof' params="id x y z roll pitch yaw update_rate gnoise">
         <!-- VL53L0X ToF sensor-->
         <link name="tof_link_${id}">
@@ -91,5 +91,5 @@
                     <topicName>gazebo/range_tof_${id}</topicName>
                     <frameName>frame_range_tof_${id}</frameName>
-                    <gaussianNoise>0.006</gaussianNoise>
+                    <gaussianNoise>${gnoise}</gaussianNoise>
                     <updateRate>${update_rate}</updateRate>
                     <radiation>light</radiation>

File: stochlite_champ/stochlite_description/urdf/stochlite.transmission.xacro (robot description, xacro)
@@ -11,112 +11,4 @@
             </actuator>
         </transmission>
-        <!-- <transmission name="fl_abd_trans">
-            <type>transmission_interface/SimpleTransmission</type>
-            <joint name="fl_abd_joint">
-                <hardwareInterface>hardware_interface/EffortJointInterface</hardwareInterface>
-            </joint>
-            <actuator name="fl_abd_motor">
-                <mechanicalReduction>1</mechanicalReduction>
-            </actuator>
-        </transmission>
-        <transmission name="fl_hip_joint_trans">
-            <type>transmission_interface/SimpleTransmission</type>
-            <joint name="fl_hip_joint">
-                <hardwareInterface>hardware_interface/EffortJointInterface</hardwareInterface>
-            </joint>
-            <actuator name="fl_hip_joint_motor">
-                <mechanicalReduction>1</mechanicalReduction>
-            </actuator>
-        </transmission>
-        <transmission name="fl_knee_joint_trans">
-            <type>transmission_interface/SimpleTransmission</type>
-            <joint name="fl_knee_joint">
-                <hardwareInterface>hardware_interface/EffortJointInterface</hardwareInterface>
-            </joint>
-            <actuator name="fl_knee_joint_motor">
-                <mechanicalReduction>1</mechanicalReduction>
-            </actuator>
-        </transmission>
-        <transmission name="fr_abd_joint_trans">
-            <type>transmission_interface/SimpleTransmission</type>
-            <joint name="fr_abd_joint">
-                <hardwareInterface>hardware_interface/EffortJointInterface</hardwareInterface>
-            </joint>
-            <actuator name="fr_abd_joint_motor">
-                <mechanicalReduction>1</mechanicalReduction>
-            </actuator>
-        </transmission>
-        <transmission name="fr_hip_joint_trans">
-            <type>transmission_interface/SimpleTransmission</type>
-            <joint name="fr_hip_joint">
-                <hardwareInterface>hardware_interface/EffortJointInterface</hardwareInterface>
-            </joint>
-            <actuator name="fr_hip_joint_motor">
-                <mechanicalReduction>1</mechanicalReduction>
-            </actuator>
-        </transmission>
-        <transmission name="fr_knee_joint_trans">
-            <type>transmission_interface/SimpleTransmission</type>
-            <joint name="fr_knee_joint">
-                <hardwareInterface>hardware_interface/EffortJointInterface</hardwareInterface>
-            </joint>
-            <actuator name="fr_knee_joint_motor">
-                <mechanicalReduction>1</mechanicalReduction>
-            </actuator>
-        </transmission>
-        <transmission name="bl_abd_trans">
-            <type>transmission_interface/SimpleTransmission</type>
-            <joint name="bl_abd_joint">
-                <hardwareInterface>hardware_interface/EffortJointInterface</hardwareInterface>
-            </joint>
-            <actuator name="bl_abd_motor">
-                <mechanicalReduction>1</mechanicalReduction>
-            </actuator>
-        </transmission>
-        <transmission name="bl_hip_joint_trans">
-            <type>transmission_interface/SimpleTransmission</type>
-            <joint name="bl_hip_joint">
-                <hardwareInterface>hardware_interface/EffortJointInterface</hardwareInterface>
-            </joint>
-            <actuator name="bl_hip_joint_motor">
-                <mechanicalReduction>1</mechanicalReduction>
-            </actuator>
-        </transmission>
-        <transmission name="bl_knee_joint_trans">
-            <type>transmission_interface/SimpleTransmission</type>
-            <joint name="bl_knee_joint">
-                <hardwareInterface>hardware_interface/EffortJointInterface</hardwareInterface>
-            </joint>
-            <actuator name="bl_knee_joint_motor">
-                <mechanicalReduction>1</mechanicalReduction>
-            </actuator>
-        </transmission>
-        <transmission name="br_abd_joint_trans">
-            <type>transmission_interface/SimpleTransmission</type>
-            <joint name="br_abd_joint">
-                <hardwareInterface>hardware_interface/EffortJointInterface</hardwareInterface>
-            </joint>
-            <actuator name="br_abd_joint_motor">
-                <mechanicalReduction>1</mechanicalReduction>
-            </actuator>
-        </transmission>
-        <transmission name="br_hip_joint_trans">
-            <type>transmission_interface/SimpleTransmission</type>
-            <joint name="br_hip_joint">
-                <hardwareInterface>hardware_interface/EffortJointInterface</hardwareInterface>
-            </joint>
-            <actuator name="br_hip_joint_motor">
-                <mechanicalReduction>1</mechanicalReduction>
-            </actuator>
-        </transmission>
-        <transmission name="br_knee_joint_trans">
-            <type>transmission_interface/SimpleTransmission</type>
-            <joint name="br_knee_joint">
-                <hardwareInterface>hardware_interface/EffortJointInterface</hardwareInterface>
-            </joint>
-            <actuator name="br_knee_joint_motor">
-                <mechanicalReduction>1</mechanicalReduction>
-            </actuator>
-        </transmission> -->
     </xacro:macro>
 </robot>

File: stochlite_champ/stochlite_description/urdf/stochlite.urdf.xacro (robot description, xacro)
@@ -40,20 +40,12 @@
     <xacro:stochlite_gazebo />
     <!-- For sensors-->
-    <xacro:imu id="1" x="0.0" y="0.0" z="0.005" roll="0.0" pitch="0.0" yaw="0.0" update_rate="20"/>
+    <xacro:imu id="1" x="0.0" y="0.0" z="0.005" roll="0.0" pitch="0.0" yaw="0.0" update_rate="20" gnoise="0.005"/>
     <!-- front triangle of tofs -->
-    <xacro:tof id="1" x="0.150" y=" 0.000" z="-0.025" roll="0.0" pitch="1.57" yaw="0.0" update_rate="20"/>
-    <xacro:tof id="2" x="0.065" y=" 0.047" z="-0.025" roll="0.0" pitch="1.57" yaw="0.0" update_rate="20"/>
-    <xacro:tof id="6" x="0.065" y="-0.047" z="-0.025" roll="0.0" pitch="1.57" yaw="0.0" update_rate="20"/>
+    <xacro:tof id="1" x="0.150" y=" 0.000" z="-0.025" roll="0.0" pitch="1.57" yaw="0.0" update_rate="20" gnoise="0.0001"/>
+    <xacro:tof id="2" x="0.065" y=" 0.047" z="-0.025" roll="0.0" pitch="1.57" yaw="0.0" update_rate="20" gnoise="0.0001"/>
+    <xacro:tof id="6" x="0.065" y="-0.047" z="-0.025" roll="0.0" pitch="1.57" yaw="0.0" update_rate="20" gnoise="0.0001"/>
     <!-- back triangle of tofs -->
-    <xacro:tof id="4" x="-0.150" y=" 0.000" z="-0.025" roll="0.0" pitch="1.57" yaw="0.0" update_rate="20"/>
-    <xacro:tof id="3" x="-0.065" y=" 0.047" z="-0.025" roll="0.0" pitch="1.57" yaw="0.0" update_rate="20"/>
-    <xacro:tof id="5" x="-0.065" y="-0.047" z="-0.025" roll="0.0" pitch="1.57" yaw="0.0" update_rate="20"/>
-    <!-- front triangle of tofs -->
-    <!-- <xacro:tof id="0" x="0.16" y=" 0.00" z="-0.025" roll="0.0" pitch="1.57" yaw="0.0" update_rate="20"/>
-    <xacro:tof id="1" x="0.06" y=" 0.055" z="-0.025" roll="0.0" pitch="1.57" yaw="0.0" update_rate="20"/>
-    <xacro:tof id="2" x="0.06" y="-0.055" z="-0.025" roll="0.0" pitch="1.57" yaw="0.0" update_rate="20"/> -->
-    <!-- back triangle of tofs -->
-    <!-- <xacro:tof id="3" x="-0.16" y=" 0.00" z="-0.025" roll="0.0" pitch="1.57" yaw="0.0" update_rate="20"/>
-    <xacro:tof id="4" x="-0.06" y=" 0.055" z="-0.025" roll="0.0" pitch="1.57" yaw="0.0" update_rate="20"/>
-    <xacro:tof id="5" x="-0.06" y="-0.055" z="-0.025" roll="0.0" pitch="1.57" yaw="0.0" update_rate="20"/> -->
+    <xacro:tof id="4" x="-0.150" y=" 0.000" z="-0.025" roll="0.0" pitch="1.57" yaw="0.0" update_rate="20" gnoise="0.0001"/>
+    <xacro:tof id="3" x="-0.065" y=" 0.047" z="-0.025" roll="0.0" pitch="1.57" yaw="0.0" update_rate="20" gnoise="0.0001"/>
+    <xacro:tof id="5" x="-0.065" y="-0.047" z="-0.025" roll="0.0" pitch="1.57" yaw="0.0" update_rate="20" gnoise="0.0001"/>
 </robot>
