Commit message: stochlite - corrected feet joint frames

File: stochlite_champ/stochlite_description/urdf/stochlite.description.xacro (robot description, xacro)
@@ -5,6 +5,6 @@
     <xacro:property name="velocity" value="4.6" />
     <xacro:property name="abd_lim" value="1.572" />
-    <xacro:property name="hip_lim" value="5.22" />
-    <xacro:property name="knee_lim" value="5.22" />
+    <xacro:property name="hip_lim" value="10.22" />
+    <xacro:property name="knee_lim" value="10.22" />
     <xacro:macro name="stochlite_description">
         <!-- For KDL -->
@@ -185,5 +185,5 @@
         </link>
         <joint name="fl_toe_joint" type="fixed">
-            <origin xyz="0 -0.023481 -0.146" rpy="0 0 0" />
+            <origin xyz="0 0.023481 -0.146" rpy="0 0 0" />
             <axis xyz="0 1 0" />
             <parent link="fl_shank_link"/>
@@ -501,5 +501,5 @@
         </link>
         <joint name="bl_toe_joint" type="fixed">
-            <origin xyz="0 -0.023481 -0.146" rpy="0 0 0" />
+            <origin xyz="0 0.023481 -0.146" rpy="0 0 0" />
             <axis xyz="0 1 0" />
             <parent link="bl_shank_link"/>

File: stochlite_champ/stochlite_description/urdf/stochlite.gazebo.xacro (robot description, xacro)
@@ -8,7 +8,7 @@
             </plugin>
         </gazebo>
-        <!-- <gazebo>
+        <gazebo>
             <self_collide>1</self_collide>
-        </gazebo> -->
+        </gazebo>
         <gazebo>
             <plugin filename="libgazebo_ros_p3d.so" name="p3d_base_controller">

File: stochlite_champ/stochlite_description/urdf/stochlite.urdf (robot description, URDF)
Before this commit: robot stochlite, 18 links, 17 joints
Joints:
- joint bl_hip_joint: limit lower=-5.22 upper=5.22 effort=4.1 velocity=4.6 -> lower=-10.22 upper=10.22 effort=4.1 velocity=4.6
- joint bl_knee_joint: limit lower=-5.22 upper=5.22 effort=4.1 velocity=4.6 -> lower=-10.22 upper=10.22 effort=4.1 velocity=4.6
- joint bl_toe_joint: origin xyz=0 -0.023481 -0.146 rpy=0 0 0 -> xyz=0 0.023481 -0.146 rpy=0 0 0
- joint br_hip_joint: limit lower=-5.22 upper=5.22 effort=4.1 velocity=4.6 -> lower=-10.22 upper=10.22 effort=4.1 velocity=4.6
- joint br_knee_joint: limit lower=-5.22 upper=5.22 effort=4.1 velocity=4.6 -> lower=-10.22 upper=10.22 effort=4.1 velocity=4.6
- joint fl_hip_joint: limit lower=-5.22 upper=5.22 effort=4.1 velocity=4.6 -> lower=-10.22 upper=10.22 effort=4.1 velocity=4.6
- joint fl_knee_joint: limit lower=-5.22 upper=5.22 effort=4.1 velocity=4.6 -> lower=-10.22 upper=10.22 effort=4.1 velocity=4.6
- joint fl_toe_joint: origin xyz=0 -0.023481 -0.146 rpy=0 0 0 -> xyz=0 0.023481 -0.146 rpy=0 0 0
- joint fr_hip_joint: limit lower=-5.22 upper=5.22 effort=4.1 velocity=4.6 -> lower=-10.22 upper=10.22 effort=4.1 velocity=4.6
- joint fr_knee_joint: limit lower=-5.22 upper=5.22 effort=4.1 velocity=4.6 -> lower=-10.22 upper=10.22 effort=4.1 velocity=4.6

Commit message: Revert "stochlite - corrected feet joint frames"
This reverts commit 12dfb949ab3766b988ba29885b55ee0770eb37df.

remove the changes in the master

File: stochlite_champ/stochlite_description/urdf/stochlite.description.xacro (robot description, xacro)
@@ -5,6 +5,6 @@
     <xacro:property name="velocity" value="4.6" />
     <xacro:property name="abd_lim" value="1.572" />
-    <xacro:property name="hip_lim" value="10.22" />
-    <xacro:property name="knee_lim" value="10.22" />
+    <xacro:property name="hip_lim" value="5.22" />
+    <xacro:property name="knee_lim" value="5.22" />
     <xacro:macro name="stochlite_description">
         <!-- For KDL -->
@@ -185,5 +185,5 @@
         </link>
         <joint name="fl_toe_joint" type="fixed">
-            <origin xyz="0 0.023481 -0.146" rpy="0 0 0" />
+            <origin xyz="0 -0.023481 -0.146" rpy="0 0 0" />
             <axis xyz="0 1 0" />
             <parent link="fl_shank_link"/>
@@ -501,5 +501,5 @@
         </link>
         <joint name="bl_toe_joint" type="fixed">
-            <origin xyz="0 0.023481 -0.146" rpy="0 0 0" />
+            <origin xyz="0 -0.023481 -0.146" rpy="0 0 0" />
             <axis xyz="0 1 0" />
             <parent link="bl_shank_link"/>

File: stochlite_champ/stochlite_description/urdf/stochlite.gazebo.xacro (robot description, xacro)
@@ -8,7 +8,7 @@
             </plugin>
         </gazebo>
-        <gazebo>
+        <!-- <gazebo>
             <self_collide>1</self_collide>
-        </gazebo>
+        </gazebo> -->
         <gazebo>
             <plugin filename="libgazebo_ros_p3d.so" name="p3d_base_controller">

File: stochlite_champ/stochlite_description/urdf/stochlite.urdf (robot description, URDF)
Before this commit: robot stochlite, 18 links, 17 joints
Joints:
- joint bl_hip_joint: limit lower=-10.22 upper=10.22 effort=4.1 velocity=4.6 -> lower=-5.22 upper=5.22 effort=4.1 velocity=4.6
- joint bl_knee_joint: limit lower=-10.22 upper=10.22 effort=4.1 velocity=4.6 -> lower=-5.22 upper=5.22 effort=4.1 velocity=4.6
- joint bl_toe_joint: origin xyz=0 0.023481 -0.146 rpy=0 0 0 -> xyz=0 -0.023481 -0.146 rpy=0 0 0
- joint br_hip_joint: limit lower=-10.22 upper=10.22 effort=4.1 velocity=4.6 -> lower=-5.22 upper=5.22 effort=4.1 velocity=4.6
- joint br_knee_joint: limit lower=-10.22 upper=10.22 effort=4.1 velocity=4.6 -> lower=-5.22 upper=5.22 effort=4.1 velocity=4.6
- joint fl_hip_joint: limit lower=-10.22 upper=10.22 effort=4.1 velocity=4.6 -> lower=-5.22 upper=5.22 effort=4.1 velocity=4.6
- joint fl_knee_joint: limit lower=-10.22 upper=10.22 effort=4.1 velocity=4.6 -> lower=-5.22 upper=5.22 effort=4.1 velocity=4.6
- joint fl_toe_joint: origin xyz=0 0.023481 -0.146 rpy=0 0 0 -> xyz=0 -0.023481 -0.146 rpy=0 0 0
- joint fr_hip_joint: limit lower=-10.22 upper=10.22 effort=4.1 velocity=4.6 -> lower=-5.22 upper=5.22 effort=4.1 velocity=4.6
- joint fr_knee_joint: limit lower=-10.22 upper=10.22 effort=4.1 velocity=4.6 -> lower=-5.22 upper=5.22 effort=4.1 velocity=4.6

Commit message: tuned PID values for joint control

File: stochlite_champ/stochlite_description/urdf/stochlite.description.xacro (robot description, xacro)
@@ -13,7 +13,7 @@
         <joint name="dummy_joint" type="fixed">
             <parent link="dummy"/>
-            <child link="base_link_torso"/>
+            <child link="base_link"/>
         </joint> -->
-        <link name="base_link_torso">
+        <link name="base_link">
             <inertial>
                 <origin xyz="0.00011698 0.00043344 -0.0081282" rpy="0 0 0" />
@@ -30,5 +30,5 @@
                 <origin xyz="0 0 0" rpy="0 0 0" />
                 <geometry>
-                    <mesh filename="package://stochlite_description/meshes/base_link_torso.STL" />
+                    <mesh filename="package://stochlite_description/meshes/base_link.STL" />
                 </geometry>
                 <material name="">
@@ -39,5 +39,5 @@
                 <origin xyz="0 0 0" rpy="0 0 0" />
                 <geometry>
-                    <mesh filename="package://stochlite_description/meshes/base_link_torso.STL" />
+                    <mesh filename="package://stochlite_description/meshes/base_link.STL" />
                 </geometry>
             </collision>
@@ -51,5 +51,5 @@
         </link>
         <joint name="imu_joint" type="fixed">
-            <parent link="base_link_torso"/>
+            <parent link="base_link"/>
             <child link="imu_link"/>
         </joint>
@@ -84,5 +84,5 @@
         <joint name="fl_abd_joint" type="revolute">
             <origin xyz="0.16695 0.0956 -0.0050001" rpy="0 0 0" />
-            <parent link="base_link_torso" />
+            <parent link="base_link" />
             <child link="fl_abd_link" />
             <axis xyz="1 0 0" />
@@ -185,5 +185,5 @@
         </link>
         <joint name="fl_toe_joint" type="fixed">
-            <origin xyz="0 0.023481 -0.146" rpy="0 0 0" />
+            <origin xyz="0 0.023481 -0.169" rpy="0 0 0" />
             <axis xyz="0 1 0" />
             <parent link="fl_shank_link"/>
@@ -231,5 +231,5 @@
         <joint name="fr_abd_joint" type="revolute">
             <origin xyz="0.16695 -0.0964 -0.0049999" rpy="0 0 0" />
-            <parent link="base_link_torso" />
+            <parent link="base_link" />
             <child link="fr_abd_link" />
             <axis xyz="1 0 0" />
@@ -343,5 +343,5 @@
         </link>
         <joint name="fr_toe_joint" type="fixed">
-            <origin xyz="0 -0.023481 -0.146" rpy="0 0 0" />
+            <origin xyz="0 -0.023481 -0.169" rpy="0 0 0" />
             <axis xyz="0 1 0" />
             <parent link="fr_shank_link"/>
@@ -389,5 +389,5 @@
         <joint name="bl_abd_joint" type="revolute">
             <origin xyz="-0.16695 0.0956 -0.0049999" rpy="0 0 0" />
-            <parent link="base_link_torso" />
+            <parent link="base_link" />
             <child link="bl_abd_link" />
             <axis xyz="1 0 0" />
@@ -501,5 +501,5 @@
         </link>
         <joint name="bl_toe_joint" type="fixed">
-            <origin xyz="0 0.023481 -0.146" rpy="0 0 0" />
+            <origin xyz="0 0.023481 -0.169" rpy="0 0 0" />
             <axis xyz="0 1 0" />
             <parent link="bl_shank_link"/>
@@ -547,5 +547,5 @@
         <joint name="br_abd_joint" type="revolute">
             <origin xyz="-0.16695 -0.0964 -0.0050001" rpy="0 0 0" />
-            <parent link="base_link_torso" />
+            <parent link="base_link" />
             <child link="br_abd_link" />
             <axis xyz="1 0 0" />
@@ -659,5 +659,5 @@
         </link>
         <joint name="br_toe_joint" type="fixed">
-            <origin xyz="0 -0.023481 -0.146" rpy="0 0 0" />
+            <origin xyz="0 -0.023481 -0.169" rpy="0 0 0" />
             <axis xyz="0 1 0" />
             <parent link="br_shank_link"/>

File: stochlite_champ/stochlite_description/urdf/stochlite.gazebo.xacro (robot description, xacro)
@@ -15,5 +15,5 @@
             <alwaysOn>true</alwaysOn>
             <updateRate>10.0</updateRate>
-            <bodyName>base_link_torso</bodyName>
+            <bodyName>base_link</bodyName>
             <topicName>odom/ground_truth</topicName>
             <gaussianNoise>0.01</gaussianNoise>

File: stochlite_champ/stochlite_description/urdf/stochlite.materials.xacro (robot description, xacro)
@@ -5,66 +5,118 @@
         <gazebo reference="base_link_torso">
             <material>Gazebo/White</material>
-            <mu1>1.0</mu1>
-            <mu2>0.5</mu2>
+            <kp>10000000.0</kp>
+            <kd>1.0</kd>
+            <mu1>4</mu1>
+            <mu2>4</mu2>
+            <maxVel>0.0</maxVel>
+            <minDepth>0.001</minDepth>
         </gazebo>
         <gazebo reference="fl_abd_link">
             <material>Gazebo/Grey</material>
-            <mu1>1.0</mu1>
-            <mu2>0.5</mu2>
+            <kp>10000000.0</kp>
+            <kd>1.0</kd>
+            <mu1>4</mu1>
+            <mu2>4</mu2>
+            <maxVel>0.0</maxVel>
+            <minDepth>0.001</minDepth>
         </gazebo>
         <gazebo reference="fl_thigh_link">
             <material>Gazebo/DarkGrey</material>
-            <mu1>1.0</mu1>
-            <mu2>0.5</mu2>
+            <kp>10000000.0</kp>
+            <kd>1.0</kd>
+            <mu1>4</mu1>
+            <mu2>4</mu2>
+            <maxVel>0.0</maxVel>
+            <minDepth>0.001</minDepth>
         </gazebo>
         <gazebo reference="fl_shank_link">
             <material>Gazebo/Grey</material>
-            <mu1>1.0</mu1>
-            <mu2>0.5</mu2>
+            <kp>10000000.0</kp>
+            <kd>1.0</kd>
+            <mu1>4</mu1>
+            <mu2>4</mu2>
+            <maxVel>0.0</maxVel>
+            <minDepth>0.001</minDepth>
         </gazebo>
         <gazebo reference="fr_abd_link">
             <material>Gazebo/Grey</material>
-            <mu1>1.0</mu1>
-            <mu2>0.5</mu2>
+            <kp>10000000.0</kp>
+            <kd>1.0</kd>
+            <mu1>4</mu1>
+            <mu2>4</mu2>
+            <maxVel>0.0</maxVel>
+            <minDepth>0.001</minDepth>
         </gazebo>
         <gazebo reference="fr_thigh_link">
             <material>Gazebo/DarkGrey</material>
-            <mu1>1.0</mu1>
-            <mu2>0.5</mu2>
+            <kp>10000000.0</kp>
+            <kd>1.0</kd>
+            <mu1>4</mu1>
+            <mu2>4</mu2>
+            <maxVel>0.0</maxVel>
+            <minDepth>0.001</minDepth>
         </gazebo>
         <gazebo reference="fr_shank_link">
             <material>Gazebo/Grey</material>
-            <mu1>1.0</mu1>
-            <mu2>0.5</mu2>
+            <kp>10000000.0</kp>
+            <kd>1.0</kd>
+            <mu1>4</mu1>
+            <mu2>4</mu2>
+            <maxVel>0.0</maxVel>
+            <minDepth>0.001</minDepth>
         </gazebo>
         <gazebo reference="bl_abd_link">
             <material>Gazebo/Grey</material>
-            <mu1>1.0</mu1>
-            <mu2>0.5</mu2>
+            <kp>10000000.0</kp>
+            <kd>1.0</kd>
+            <mu1>4</mu1>
+            <mu2>4</mu2>
+            <maxVel>0.0</maxVel>
+            <minDepth>0.001</minDepth>
         </gazebo>
         <gazebo reference="bl_thigh_link">
             <material>Gazebo/DarkGrey</material>
-            <mu1>1.0</mu1>
-            <mu2>0.5</mu2>
+            <kp>10000000.0</kp>
+            <kd>1.0</kd>
+            <mu1>4</mu1>
+            <mu2>4</mu2>
+            <maxVel>0.0</maxVel>
+            <minDepth>0.001</minDepth>
         </gazebo>
         <gazebo reference="bl_shank_link">
             <material>Gazebo/Grey</material>
-            <mu1>1.0</mu1>
-            <mu2>0.5</mu2>
+            <kp>10000000.0</kp>
+            <kd>1.0</kd>
+            <mu1>4</mu1>
+            <mu2>4</mu2>
+            <maxVel>0.0</maxVel>
+            <minDepth>0.001</minDepth>
         </gazebo>
         <gazebo reference="br_abd_link">
             <material>Gazebo/Grey</material>
-            <mu1>1.0</mu1>
-            <mu2>0.5</mu2>
+            <kp>10000000.0</kp>
+            <kd>1.0</kd>
+            <mu1>4</mu1>
+            <mu2>4</mu2>
+            <maxVel>0.0</maxVel>
+            <minDepth>0.001</minDepth>
         </gazebo>
         <gazebo reference="br_thigh_link">
             <material>Gazebo/DarkGrey</material>
-            <mu1>1.0</mu1>
-            <mu2>0.5</mu2>
+            <kp>10000000.0</kp>
+            <kd>1.0</kd>
+            <mu1>4</mu1>
+            <mu2>4</mu2>
+            <maxVel>0.0</maxVel>
+            <minDepth>0.001</minDepth>
         </gazebo>
         <gazebo reference="br_shank_link">
             <material>Gazebo/Grey</material>
-            <mu1>1.0</mu1>
-            <mu2>0.5</mu2>
+            <kp>10000000.0</kp>
+            <kd>1.0</kd>
+            <mu1>4</mu1>
+            <mu2>4</mu2>
+            <maxVel>0.0</maxVel>
+            <minDepth>0.001</minDepth>
         </gazebo>
     </xacro:macro>

File: stochlite_champ/stochlite_description/urdf/stochlite.urdf (robot description, URDF)
Before this commit: robot stochlite, 18 links, 17 joints
Links:
- removed link base_link_torso
- added link base_link, mass 1.582; collision mesh filename=package://stochlite_description/meshes/base_link.STL; visual mesh filename=package://stochlite_description/meshes/base_link.STL
Joints:
- joint bl_abd_joint: parent base_link_torso -> base_link
- joint bl_toe_joint: origin xyz=0 0.023481 -0.146 rpy=0 0 0 -> xyz=0 0.023481 -0.169 rpy=0 0 0
- joint br_abd_joint: parent base_link_torso -> base_link
- joint br_toe_joint: origin xyz=0 -0.023481 -0.146 rpy=0 0 0 -> xyz=0 -0.023481 -0.169 rpy=0 0 0
- joint fl_abd_joint: parent base_link_torso -> base_link
- joint fl_toe_joint: origin xyz=0 0.023481 -0.146 rpy=0 0 0 -> xyz=0 0.023481 -0.169 rpy=0 0 0
- joint fr_abd_joint: parent base_link_torso -> base_link
- joint fr_toe_joint: origin xyz=0 -0.023481 -0.146 rpy=0 0 0 -> xyz=0 -0.023481 -0.169 rpy=0 0 0
- joint imu_joint: parent base_link_torso -> base_link

Commit message: added VL53L0X tof sensor

File: stochlite_champ/stochlite_description/urdf/stochlite.description.xacro (robot description, xacro)
@@ -43,15 +43,4 @@
             </collision>
         </link>
-        <link name="imu_link">
-            <inertial>
-            <mass value="0.001"/>
-            <origin rpy="0 0 0" xyz="0 0 0"/>
-            <inertia ixx="1e-09" ixy="0.0" ixz="0.0" iyy="1e-09" iyz="0.0" izz="1e-09"/>
-            </inertial>
-        </link>
-        <joint name="imu_joint" type="fixed">
-            <parent link="base_link"/>
-            <child link="imu_link"/>
-        </joint>
         <link name="fl_abd_link">
             <inertial>

File: stochlite_champ/stochlite_description/urdf/stochlite.gazebo.xacro (robot description, xacro)
@@ -13,26 +13,63 @@
         <gazebo>
             <plugin filename="libgazebo_ros_p3d.so" name="p3d_base_controller">
-            <alwaysOn>true</alwaysOn>
-            <updateRate>10.0</updateRate>
-            <bodyName>base_link</bodyName>
-            <topicName>odom/ground_truth</topicName>
-            <gaussianNoise>0.01</gaussianNoise>
-            <frameName>world</frameName>
-            <xyzOffsets>0 0 0</xyzOffsets>
-            <rpyOffsets>0 0 0</rpyOffsets>
+                <alwaysOn>true</alwaysOn>
+                <updateRate>10.0</updateRate>
+                <bodyName>base_link</bodyName>
+                <topicName>odom/ground_truth</topicName>
+                <gaussianNoise>0.01</gaussianNoise>
+                <frameName>world</frameName>
+                <xyzOffsets>0 0 0</xyzOffsets>
+                <rpyOffsets>0 0 0</rpyOffsets>
             </plugin>
         </gazebo>
         <gazebo>
             <plugin filename="libhector_gazebo_ros_imu.so" name="imu_controller">
-            <updateRate>50.0</updateRate>
-            <bodyName>imu_link</bodyName>
-            <topicName>imu/data</topicName>
-            <accelDrift>0.005 0.005 0.005</accelDrift>
-            <accelGaussianNoise>0.005 0.005 0.005</accelGaussianNoise>
-            <rateDrift>0.005 0.005 0.005 </rateDrift>
-            <rateGaussianNoise>0.005 0.005 0.005 </rateGaussianNoise>
-            <headingDrift>0.005</headingDrift>
-            <headingGaussianNoise>0.005</headingGaussianNoise>
+                <updateRate>50.0</updateRate>
+                <bodyName>imu_link</bodyName>
+                <topicName>imu/data</topicName>
+                <accelDrift>0.005 0.005 0.005</accelDrift>
+                <accelGaussianNoise>0.005 0.005 0.005</accelGaussianNoise>
+                <rateDrift>0.005 0.005 0.005 </rateDrift>
+                <rateGaussianNoise>0.005 0.005 0.005 </rateGaussianNoise>
+                <headingDrift>0.005</headingDrift>
+                <headingGaussianNoise>0.005</headingGaussianNoise>
             </plugin>
+        </gazebo>
+        <gazebo reference="tof_link">
+            <sensor type="ray" name="tof_sensor">
+                <visualize>true</visualize>
+                <update_rate>70</update_rate>
+                <always_on>1</always_on>
+                <ray>
+                    <scan>
+                        <horizontal>
+                            <samples>10</samples>
+                            <resolution>2</resolution>
+                            <min_angle>-0.02618</min_angle>
+                            <max_angle>0.02618</max_angle>
+                        </horizontal>
+                        <vertical>
+                            <samples>10</samples>
+                            <resolution>2</resolution>
+                            <min_angle>-0.02618</min_angle>
+                            <max_angle>0.02618</max_angle>
+                        </vertical>
+                    </scan>
+                    <range>
+                        <min>0.02</min>
+                        <max>2</max>
+                        <!-- <radius>0.33974388395</radius> -->
+                        <resolution>0.05</resolution>
+                    </range>
+                </ray>
+                <plugin name="tof_plugin" filename="libgazebo_ros_range.so">
+                    <topicName>gazebo/range_tof</topicName>
+                    <frameName>range_tof_map</frameName>
+                    <gaussianNoise>0.06</gaussianNoise>
+                    <updateRate>70</updateRate>
+                    <radiation>light</radiation>
+                    <fov>0.43</fov>
+                </plugin>
+            </sensor>
         </gazebo>
     </xacro:macro>

File: stochlite_champ/stochlite_description/urdf/stochlite.materials.xacro (robot description, xacro)
@@ -120,4 +120,10 @@
             <minDepth>0.001</minDepth>
         </gazebo>
+        <gazebo reference="tof_link">
+            <material>Gazebo/Red</material>
+        </gazebo>
+        <gazebo reference="imu_link">
+            <material>Gazebo/Yellow</material>
+        </gazebo>
     </xacro:macro>
 </robot>

File: stochlite_champ/stochlite_description/urdf/stochlite.urdf (robot description, URDF)
Before this commit: robot stochlite, 18 links, 17 joints
Links:
- added link tof_link, mass 0.001; visual box size=0.005 0.015 0.005
- link imu_link: geometry visual box size=0.005 0.005 0.005
Joints:
- added joint tof_joint: type fixed, parent base_link, child tof_link, origin xyz=0 0 -0.029 rpy=0 1.57 0
- joint imu_joint: origin (none) -> xyz=0 0 0.005 rpy=0 0 0

File: stochlite_champ/stochlite_description/urdf/stochlite.urdf.xacro (robot description, xacro)
@@ -1,2 +1,3 @@
+<?xml version="1.0" encoding="utf-8"?>
 <robot name = 'stochlite' xmlns:xacro = 'http://www.ros.org/wiki/xacro'>
     <xacro:include filename="$(find stochlite_description)/urdf/stochlite.description.xacro" />
@@ -4,5 +5,11 @@
     <xacro:include filename="$(find stochlite_description)/urdf/stochlite.gazebo.xacro" />
     <xacro:include filename="$(find stochlite_description)/urdf/stochlite.materials.xacro" />
+    <xacro:include filename="$(find stochlite_description)/urdf/stochlite.sensors.xacro" />
+    <!-- <xacro:include filename="$(find teraranger_description)/urdf/base_hub.urdf.xacro"/> -->
+    <!-- <xacro:include filename="$(find teraranger_description)/urdf/teraranger_one.urdf.xacro"/>     -->
     <xacro:stochlite_description />
+    <xacro:stochlite_sensors />
+    <!-- <xacro:base_hub multi_hub="0" hub_id="0" parent="base_link" x="0" y="0.000" z="-0.029" roll="0.0" pitch="0.0" yaw="0.0"/> -->
+    <!-- <xacro:teraranger_one multi_hub="0" hub_id="0" id="0" x="0" y="0.000" z="0.000" roll="0.0" pitch="1.57" yaw="0.0" gaussian_noise="0.06"/> -->
     <xacro:stochlite_transmission />
     <xacro:stochlite_gazebo />
