Commit message: Added urdf for fixed motion
-changed the pid values and commited the old ones
-added argument for spwaning it at a hight
-Trot gait file the step length has been forced to 0

File: stochlite_champ/stochlite_description/urdf/stochlite.description.xacro (robot description, xacro)
@@ -9,10 +9,10 @@
     <xacro:macro name="stochlite_description">
         <!-- For KDL -->
-        <!-- <link name="dummy">
-        </link>
-        <joint name="dummy_joint" type="fixed">
-            <parent link="dummy"/>
+        <link name="world">
+        </link>
+        <joint name="fixed" type="fixed">
+            <parent link="world"/>
             <child link="base_link"/>
-        </joint> -->
+        </joint>
         <link name="base_link">
             <inertial>
